File: hardware/kicad/msx-joydolphin-v2-Build1b/msx-joydolphin-v2.kicad_pcb (KiCad board)
At the start: 2 copper layers, 55 x 32 mm, 20 parts, among them J1 J2 GCN, J2 J1 MSX, J3 DEBUG, Q1 BSS138, U1 74LS03, U2 74LS03

Commit message: v2-build1c: prototype built
Signed-off-by: Albert Herranz <albert_herranz@yahoo.es>
Other:
- outline, holes or cut-outs redrawn
Changed lines of the file:
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@@
       (plot_on_all_layers_selection 0x0000000_00000000)
       (disableapertmacros false)
-      (usegerberextensions true)
+      (usegerberextensions false)
       (usegerberattributes false)
       (usegerberadvancedattributes false)
@@
     (property "ki_description" "Resistor")
     (property "ki_keywords" "R res resistor")
-    (attr smd)
+    (attr smd exclude_from_bom)
     (fp_text reference "R3" (at 3.45 0) (layer "B.SilkS")
         (effects (font (size 0.8 1) (thickness 0.15)) (justify mirror))
@@
         (effects (font (size 1 1) (thickness 0.15)) (justify mirror))
     )
-    (fp_text value "74LS03" (at -4.175 2.39 180) (layer "B.SilkS")
+    (fp_text value "74LS03" (at -4.175 2.39) (layer "B.SilkS")
         (effects (font (size 0.8 0.8) (thickness 0.15)) (justify mirror))
     )
@@
     (fp_line (start 0 -4.435) (end 1.95 -4.435)
       (stroke (width 0.12) (type solid)) (layer "B.SilkS"))
-    (fp_line (start 0 4.435) (end -3.45 4.435)
+    (fp_line (start 0 4.435) (end -1.95 4.435)
       (stroke (width 0.12) (type solid)) (layer "B.SilkS"))
     (fp_line (start 0 4.435) (end 1.95 4.435)
       (stroke (width 0.12) (type solid)) (layer "B.SilkS"))
+    (fp_poly
+      (pts
+        (xy -2.7 4.37)
+        (xy -2.94 4.7)
+        (xy -2.46 4.7)
+        (xy -2.7 4.37)
+      )
+      (stroke (width 0.12) (type solid)) (fill solid) (layer "B.SilkS"))
     (fp_line (start -3.7 -4.58) (end 3.7 -4.58)
       (stroke (width 0.05) (type solid)) (layer "B.CrtYd"))
@@
     (pad "14" smd roundrect (at 2.475 3.81 270) (size 1.95 0.6) (layers "B.Cu" "B.Paste" "B.Mask") (roundrect_rratio 0.25)
       (net 27 "/VCC_5V") (pinfunction "VCC") (pintype "power_in"))
-    (model "${KICAD6_3DMODEL_DIR}/Package_SO.3dshapes/SOIC-14_3.9x8.7mm_P1.27mm.wrl"
+    (model "${KICAD7_3DMODEL_DIR}/Package_SO.3dshapes/SOIC-14_3.9x8.7mm_P1.27mm.wrl"
       (offset (xyz 0 0 0))
       (scale (xyz 1 1 1))
@@
     (fp_line (start 0 -1.56) (end 0.65 -1.56)
       (stroke (width 0.12) (type solid)) (layer "B.SilkS"))
-    (fp_line (start 0 1.56) (end -1.675 1.56)
+    (fp_line (start 0 1.56) (end -0.65 1.56)
       (stroke (width 0.12) (type solid)) (layer "B.SilkS"))
     (fp_line (start 0 1.56) (end 0.65 1.56)
       (stroke (width 0.12) (type solid)) (layer "B.SilkS"))
+    (fp_poly
+      (pts
+        (xy -1.1625 1.51)
+        (xy -1.4025 1.84)
+        (xy -0.9225 1.84)
+        (xy -1.1625 1.51)
+      )
+      (stroke (width 0.12) (type solid)) (fill solid) (layer "B.SilkS"))
     (fp_line (start -1.92 -1.7) (end 1.92 -1.7)
       (stroke (width 0.05) (type solid)) (layer "B.CrtYd"))
@@
     (pad "3" smd roundrect (at 0.9375 0 180) (size 1.475 0.6) (layers "B.Cu" "B.Paste" "B.Mask") (roundrect_rratio 0.25)
       (net 10 "/GCN_DATA_5V") (pinfunction "D") (pintype "passive"))
-    (model "${KICAD6_3DMODEL_DIR}/Package_TO_SOT_SMD.3dshapes/SOT-23.wrl"
+    (model "${KICAD7_3DMODEL_DIR}/Package_TO_SOT_SMD.3dshapes/SOT-23.wrl"
       (offset (xyz 0 0 0))
       (scale (xyz 1 1 1))
@@
     (fp_line (start 0 -4.435) (end 1.95 -4.435)
       (stroke (width 0.12) (type solid)) (layer "B.SilkS"))
-    (fp_line (start 0 4.435) (end -3.45 4.435)
+    (fp_line (start 0 4.435) (end -1.95 4.435)
       (stroke (width 0.12) (type solid)) (layer "B.SilkS"))
     (fp_line (start 0 4.435) (end 1.95 4.435)
       (stroke (width 0.12) (type solid)) (layer "B.SilkS"))
+    (fp_poly
+      (pts
+        (xy -2.7 4.37)
+        (xy -2.94 4.7)
+        (xy -2.46 4.7)
+        (xy -2.7 4.37)
+      )
+      (stroke (width 0.12) (type solid)) (fill solid) (layer "B.SilkS"))
     (fp_line (start -3.7 -4.58) (end 3.7 -4.58)
       (stroke (width 0.05) (type solid)) (layer "B.CrtYd"))
@@
     (pad "14" smd roundrect (at 2.475 3.81 90) (size 1.95 0.6) (layers "B.Cu" "B.Paste" "B.Mask") (roundrect_rratio 0.25)
       (net 27 "/VCC_5V") (pinfunction "VCC") (pintype "power_in"))
-    (model "${KICAD6_3DMODEL_DIR}/Package_SO.3dshapes/SOIC-14_3.9x8.7mm_P1.27mm.wrl"
+    (model "${KICAD7_3DMODEL_DIR}/Package_SO.3dshapes/SOIC-14_3.9x8.7mm_P1.27mm.wrl"
       (offset (xyz 0 0 0))
       (scale (xyz 1 1 1))
@@
   (gr_line (start 57.781493 63.863657) (end 57.761804 63.833728)
     (stroke (width 0.079472) (type solid)) (layer "F.SilkS"))
-  (gr_rect (start 42 36.5) (end 97 68.5)
-    (stroke (width 0.1) (type default)) (fill none) (layer "Edge.Cuts"))
+  (gr_line (start 44.5 36.5) (end 94.5 36.5)
+    (stroke (width 0.1) (type default)) (layer "Edge.Cuts"))
+  (gr_line (start 94.5 68.5) (end 44.5 68.5)
+    (stroke (width 0.1) (type default)) (layer "Edge.Cuts"))
+  (gr_arc (start 94.5 36.5) (mid 96.267767 37.232233) (end 97 39)
+    (stroke (width 0.1) (type default)) (layer "Edge.Cuts"))
+  (gr_line (start 97 39) (end 97 66)
+    (stroke (width 0.1) (type default)) (layer "Edge.Cuts"))
+  (gr_arc (start 44.5 68.5) (mid 42.732233 67.767767) (end 42 66)
+    (stroke (width 0.1) (type default)) (layer "Edge.Cuts"))
+  (gr_arc (start 97 66) (mid 96.267767 67.767767) (end 94.5 68.5)
+    (stroke (width 0.1) (type default)) (layer "Edge.Cuts"))
+  (gr_arc (start 42 39) (mid 42.732233 37.232233) (end 44.5 36.5)
+    (stroke (width 0.1) (type default)) (layer "Edge.Cuts"))
+  (gr_line (start 42 66) (end 42 39)
+    (stroke (width 0.1) (type default)) (layer "Edge.Cuts"))
   (gr_text "OUT" (at 74.5 62.3) (layer "B.SilkS")
     (effects (font (size 0.8 0.8) (thickness 0.2)) (justify mirror))
