File: hardware/kicad/msx-joydolphin-v2-Build1b/msx-joydolphin-v2.kicad_sch (KiCad schematic)
At the start: 20 parts, among them J1 J2 GCN, J2 J1 MSX, J3 DEBUG, Q1 BSS138, U1 74LS03, U2 74LS03

Commit message: v2-build1c: prototype built
Signed-off-by: Albert Herranz <albert_herranz@yahoo.es>
Parts:
- R3: now left out of the parts list
Changed lines of the file:
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@@
   )
   (symbol (lib_id "Device:R") (at 153.67 182.88 0) (unit 1)
-    (in_bom yes) (on_board yes) (dnp no) (fields_autoplaced)
+    (in_bom no) (on_board yes) (dnp no) (fields_autoplaced)
     (property "Reference" "R3" (at 156.21 181.61 0)
       (effects (font (size 1.27 1.27)) (justify left))
